File: single_driver LTC6992/single_driver LTC6992.kicad_pcb (KiCad board)
At the start: 2 copper layers, 40 parts, among them J1 Conn_02x02_Counter_Clockwise, J2 Screw_Terminal_01x02, J3 Conn_01x08_Male, SW1 SW_DIP_x06, U1 LTC6992-1 (Rev. D), U2 LM7805_TO220, U3 DRV10970

Commit message: Basically finished pcb
Parts:
- moved J2 38.9 mm to (162.9, 99.8), turned to 90 degrees
- moved J3 20.3 mm to (125.5, 95.8), turned to 180 degrees
- moved C6 6.89 mm to (150.5, 94.1), turned to 90 degrees
- moved RV1 6.74 mm to (153.7, 105.8)
- moved C9 5.00 mm to (133.7, 87.9)
- moved R5 2.85 mm to (153.1, 87.9)
- moved C2 2.29 mm to (153.3, 90.4)
- moved C4 2.29 mm to (153.3, 92.5)
- moved R15 2.29 mm to (158.6, 91.9)
- moved R9 2.29 mm to (133.8, 79.5)
- moved R6 2.16 mm to (149.4, 87.4)
- moved R2 2.16 mm to (133.8, 85.5)
- moved C1 2.05 mm to (159.4, 88.4)
- moved C5 2.05 mm to (156.8, 88.4)
- moved R11 2.03 mm to (133.8, 83.6)
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Routing:
- net /VINT: track 0.00 -> 104.3 mm, vias 0 -> 5
- net +5V: track 61.4 -> 143.1 mm, vias 0 -> 5
- net /FR: track 0.00 -> 61.1 mm
- net +12V: track 0.00 -> 55.8 mm, vias 0 -> 1
- net /DAA: track 0.00 -> 51.9 mm, vias 0 -> 1
- net /CMTMOD: track 0.00 -> 48.4 mm, vias 0 -> 2
- net /FG: track 0.00 -> 42.6 mm, vias 0 -> 3
- net /BRKMOD: track 7.39 -> 45.5 mm, vias 0 -> 2
- net /RD: track 0.00 -> 34.4 mm, vias 0 -> 2
- net Net-(J3-Pad1): track 0.00 -> 33.0 mm, vias 0 -> 1
- net /HBIAS: track 0.00 -> 31.7 mm
- net Net-(J3-Pad2): track 0.00 -> 27.0 mm, vias 0 -> 1
- net GND: track 1.36 -> 27.2 mm, vias 19 -> 21
- net /HV: track 0.00 -> 21.6 mm, vias 0 -> 1
- net /HU: track 0.00 -> 17.5 mm, vias 0 -> 2
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- added copper zone on B.Cu, net GND

Commit message: Finished...?
Parts:
- added REF**: MountingHole_3.2mm_M3, MountingHole:MountingHole_3.2mm_M3, F.Cu at (119.5, 72.5)
- added REF**: MountingHole_3.2mm_M3, MountingHole:MountingHole_3.2mm_M3, F.Cu at (119.5, 108.1)
- added REF**: MountingHole_3.2mm_M3, MountingHole:MountingHole_3.2mm_M3, F.Cu at (167.6, 108.1)
- added REF**: MountingHole_3.2mm_M3, MountingHole:MountingHole_3.2mm_M3, F.Cu at (167.6, 72.6)
Routing:
- net +12V: track 55.8 -> 57.1 mm
- net GND: track 27.2 -> 28.2 mm
Other:
- board outline added: 58.9 x 47 mm
Changed lines of the file:
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@@
   (general
     (thickness 1.6)
-    (drawings 0)
-    (tracks 482)
+    (drawings 8)
+    (tracks 492)
     (zones 0)
-    (modules 40)
+    (modules 44)
     (nets 34)
   )
@@
     (add_net "Net-(R6-Pad1)")
   )
+  (module MountingHole:MountingHole_3.2mm_M3 (layer F.Cu)
+    (at 119.507 72.517)
+    (descr "Mounting Hole 3.2mm, no annular, M3")
+    (tags "mounting hole 3.2mm no annular m3")
+    (attr virtual)
+    (fp_text reference REF** (at 0 -4.2) (layer F.SilkS)
+      (effects (font (size 1 1) (thickness 0.15)))
+    )
+    (fp_text value MountingHole_3.2mm_M3 (at 0 4.2) (layer F.Fab)
+      (effects (font (size 1 1) (thickness 0.15)))
+    )
+    (fp_circle (center 0 0) (end 3.45 0) (layer F.CrtYd) (width 0.05))
+    (fp_circle (center 0 0) (end 3.2 0) (layer Cmts.User) (width 0.15))
+    (fp_text user %R (at 0.3 0) (layer F.Fab)
+      (effects (font (size 1 1) (thickness 0.15)))
+    )
+    (pad 1 np_thru_hole circle (at 0 0) (size 3.2 3.2) (drill 3.2) (layers *.Cu *.Mask))
+  )
+  (module MountingHole:MountingHole_3.2mm_M3 (layer F.Cu)
+    (at 119.507 108.077)
+    (descr "Mounting Hole 3.2mm, no annular, M3")
+    (tags "mounting hole 3.2mm no annular m3")
+    (attr virtual)
+    (fp_text reference REF** (at 0 -4.2) (layer F.SilkS)
+      (effects (font (size 1 1) (thickness 0.15)))
+    )
+    (fp_text value MountingHole_3.2mm_M3 (at 0 4.2) (layer F.Fab)
+      (effects (font (size 1 1) (thickness 0.15)))
+    )
+    (fp_text user %R (at 0.3 0) (layer F.Fab)
+      (effects (font (size 1 1) (thickness 0.15)))
+    )
+    (fp_circle (center 0 0) (end 3.2 0) (layer Cmts.User) (width 0.15))
+    (fp_circle (center 0 0) (end 3.45 0) (layer F.CrtYd) (width 0.05))
+    (pad 1 np_thru_hole circle (at 0 0) (size 3.2 3.2) (drill 3.2) (layers *.Cu *.Mask))
+  )
+  (module MountingHole:MountingHole_3.2mm_M3 (layer F.Cu)
+    (at 167.64 108.077)
+    (descr "Mounting Hole 3.2mm, no annular, M3")
+    (tags "mounting hole 3.2mm no annular m3")
+    (attr virtual)
+    (fp_text reference REF** (at 0 -4.2) (layer F.SilkS)
+      (effects (font (size 1 1) (thickness 0.15)))
+    )
+    (fp_text value MountingHole_3.2mm_M3 (at 0 4.2) (layer F.Fab)
+      (effects (font (size 1 1) (thickness 0.15)))
+    )
+    (fp_circle (center 0 0) (end 3.45 0) (layer F.CrtYd) (width 0.05))
+    (fp_circle (center 0 0) (end 3.2 0) (layer Cmts.User) (width 0.15))
+    (fp_text user %R (at 0.3 0) (layer F.Fab)
+      (effects (font (size 1 1) (thickness 0.15)))
+    )
+    (pad 1 np_thru_hole circle (at 0 0) (size 3.2 3.2) (drill 3.2) (layers *.Cu *.Mask))
+  )
+  (module MountingHole:MountingHole_3.2mm_M3 (layer F.Cu)
+    (at 167.64 72.644)
+    (descr "Mounting Hole 3.2mm, no annular, M3")
+    (tags "mounting hole 3.2mm no annular m3")
+    (attr virtual)
+    (fp_text reference REF** (at 0 -4.2) (layer F.SilkS)
+      (effects (font (size 1 1) (thickness 0.15)))
+    )
+    (fp_text value MountingHole_3.2mm_M3 (at 0 4.2) (layer F.Fab)
+      (effects (font (size 1 1) (thickness 0.15)))
+    )
+    (fp_text user %R (at 0.3 0) (layer F.Fab)
+      (effects (font (size 1 1) (thickness 0.15)))
+    )
+    (fp_circle (center 0 0) (end 3.2 0) (layer Cmts.User) (width 0.15))
+    (fp_circle (center 0 0) (end 3.45 0) (layer F.CrtYd) (width 0.05))
+    (pad 1 np_thru_hole circle (at 0 0) (size 3.2 3.2) (drill 3.2) (layers *.Cu *.Mask))
+  )
   (module Resistor_SMD:R_0603_1608Metric (layer F.Cu)
     (at 133.795 79.502 180)
@@
     (descr "TO-220-3, Vertical, RM 2.54mm, see https://www.vishay.com/docs/66542/to-220-1.pdf")
     (tags "TO-220-3 Vertical RM 2.54mm")
-    (fp_text reference U2 (at 2.54 -4.27) (layer F.SilkS)
+    (fp_text reference U2 (at 2.54 -3.937) (layer F.SilkS)
       (effects (font (size 1 1) (thickness 0.15)))
     )
@@
     )
   )
+  (gr_line (start 168.529 67.056) (end 118.491 67.056) (layer Edge.Cuts) (width 0.05))
+  (gr_line (start 172.974 109.728) (end 172.847 71.374) (layer Edge.Cuts) (width 0.05))
+  (gr_line (start 118.364 113.665) (end 168.656 114.046) (layer Edge.Cuts) (width 0.05))
+  (gr_line (start 114.173 71.374) (end 114.046 109.347) (layer Edge.Cuts) (width 0.05))
+  (gr_arc (start 168.529 71.374) (end 172.847 71.374) (angle -90) (layer Edge.Cuts) (width 0.05))
+  (gr_arc (start 118.491 71.374) (end 118.491 67.056) (angle -90) (layer Edge.Cuts) (width 0.05))
+  (gr_arc (start 118.364 109.347) (end 114.046 109.347) (angle -90) (layer Edge.Cuts) (width 0.05))
+  (gr_arc (start 168.656 109.728) (end 168.656 114.046) (angle -90) (layer Edge.Cuts) (width 0.05))
   (via (at 129.794 89.916) (size 0.8) (drill 0.4) (layers F.Cu B.Cu) (net 2))
   (via (at 127.508 91.44) (size 0.8) (drill 0.4) (layers F.Cu B.Cu) (net 2))
@@
   (segment (start 167.40201 79.479012) (end 167.125022 79.756) (width 0.25) (layer F.Cu) (net 2))
   (segment (start 167.40201 79.032988) (end 167.40201 79.479012) (width 0.25) (layer F.Cu) (net 2))
-  (segment (start 164.569022 76.2) (end 167.40201 79.032988) (width 0.25) (layer F.Cu) (net 2))
-  (segment (start 161.544 76.2) (end 164.569022 76.2) (width 0.25) (layer F.Cu) (net 2))
   (segment (start 139.7 83.82) (end 141.224 85.344) (width 0.25) (layer F.Cu) (net 2))
   (segment (start 139.7 79.248) (end 139.7 83.82) (width 0.25) (layer F.Cu) (net 2))
@@
   (segment (start 138.3615 88.919) (end 139.149 88.919) (width 0.25) (layer F.Cu) (net 2))
   (segment (start 129.919001 96.795001) (end 132.459001 94.255001) (width 0.25) (layer B.Cu) (net 2))
+  (segment (start 166.9759 78.80599) (end 166.475899 78.305989) (width 0.25) (layer F.Cu) (net 2))
+  (segment (start 167.175012 78.80599) (end 166.9759 78.80599) (width 0.25) (layer F.Cu) (net 2))
+  (segment (start 167.40201 79.032988) (end 167.175012 78.80599) (width 0.25) (layer F.Cu) (net 2))
+  (segment (start 166.475899 78.305989) (end 161.871989 78.305989) (width 0.25) (layer F.Cu) (net 2))
+  (segment (start 161.544 77.978) (end 161.544 76.2) (width 0.25) (layer F.Cu) (net 2))
+  (segment (start 161.871989 78.305989) (end 161.544 77.978) (width 0.25) (layer F.Cu) (net 2))
   (segment (start 141.984999 76.328001) (end 142.367 75.946) (width 0.25) (layer F.Cu) (net 3))
   (segment (start 141.984999 77.471001) (end 141.984999 76.328001) (width 0.25) (layer F.Cu) (net 3))
   (segment (start 141.984999 77.989999) (end 143.243 79.248) (width 0.25) (layer F.Cu) (net 3))
   (segment (start 141.984999 77.471001) (end 141.984999 77.989999) (width 0.25) (layer F.Cu) (net 3))
-  (segment (start 167.852019 78.846587) (end 162.415412 73.40998) (width 0.25) (layer F.Cu) (net 3))
-  (segment (start 167.852019 94.910981) (end 167.852019 78.846587) (width 0.25) (layer F.Cu) (net 3))
-  (segment (start 162.941 99.822) (end 167.852019 94.910981) (width 0.25) (layer F.Cu) (net 3))
-  (segment (start 162.415412 73.40998) (end 148.07802 73.40998) (width 0.25) (layer F.Cu) (net 3))
   (segment (start 148.07802 73.40998) (end 148.07802 73.40998) (width 0.25) (layer F.Cu) (net 3))
   (via (at 148.07802 73.40998) (size 0.8) (drill 0.4) (layers F.Cu B.Cu) (net 3))
   (segment (start 144.90302 73.40998) (end 142.367 75.946) (width 0.25) (layer B.Cu) (net 3))
   (segment (start 148.07802 73.40998) (end 144.90302 73.40998) (width 0.25) (layer B.Cu) (net 3))
+  (segment (start 160.91298 73.40998) (end 148.07802 73.40998) (width 0.25) (layer F.Cu) (net 3))
+  (segment (start 162.433 74.93) (end 160.91298 73.40998) (width 0.25) (layer F.Cu) (net 3))
+  (segment (start 162.433 77.216) (end 162.433 74.93) (width 0.25) (layer F.Cu) (net 3))
+  (segment (start 163.072979 77.855979) (end 162.433 77.216) (width 0.25) (layer F.Cu) (net 3))
+  (segment (start 166.662299 77.855979) (end 163.072979 77.855979) (width 0.25) (layer F.Cu) (net 3))
+  (segment (start 167.162301 78.355981) (end 166.662299 77.855979) (width 0.25) (layer F.Cu) (net 3))
+  (segment (start 167.361413 78.355981) (end 167.162301 78.355981) (width 0.25) (layer F.Cu) (net 3))
+  (segment (start 167.852019 78.846587) (end 167.361413 78.355981) (width 0.25) (layer F.Cu) (net 3))
+  (segment (start 167.852019 94.910981) (end 167.852019 78.846587) (width 0.25) (layer F.Cu) (net 3))
+  (segment (start 162.941 99.822) (end 167.852019 94.910981) (width 0.25) (layer F.Cu) (net 3))
   (segment (start 144.018 108.458) (end 142.494 109.982) (width 0.25) (layer F.Cu) (net 4))
   (segment (start 138.938 108.458) (end 137.414 109.982) (width 0.25) (layer F.Cu) (net 4))
@@
     (polygon
       (pts
-        (xy 169.037 112.268) (xy 120.65 112.268) (xy 120.65 71.12) (xy 169.037 71.12)
+        (xy 169.037 101.6) (xy 121.666 101.727) (xy 121.666 71.12) (xy 169.037 71.12)
       )
     )
