File: pwm_dac_LTC6992/pwm_dac_LTC6992/pwm_dac_LTC6992.sch (KiCad schematic (older format))
At the start: 13 parts, among them J2 Screw_Terminal_01x03, U1 LTC6992-1 (Rev. D)

Commit message: More PWM dac stuffff
Parts:
- added J3: Conn_01x08_Male, Connector_PinHeader_2.54mm:PinHeader_1x08_P2.54mm_Vertical, symbol Connector:Conn_01x08_Male
- added R18, R19, R20, R21: 100k, Resistor_SMD:R_0603_1608Metric, symbol Device:R_Small
- added SW1: SW_DIP_x06, HS2_parts:DIP762W56P254L1772H585Q12, symbol 1825057-5:1825057-5
- J2: value Screw_Terminal_01x03 -> Screw_Terminal_01x02; symbol Connector:Screw_Terminal_01x03 -> Connector:Screw_Terminal_01x02
Connections:
- net GND: now also R18.1, R19.1, R20.1, R21.1
- net PWM: no longer J2.3 (Pin_3)
- new net: R20.2, SW1.10, SW1.9
- new net: R21.2, SW1.7, SW1.8
- new net BRKMOD: R18.2, SW1.12
- new net CMTMOD: SW1.3
- new net DAA: SW1.5
- new net FR: R19.2, SW1.11
- new net VINT: SW1.1, SW1.2, SW1.4, SW1.6
Changed lines of the file:
@@
 	4800 3800 4800 3750
-$Comp
-L power:+5V #PWR0115
-U 1 1 5FA557E2
-P 5150 2000
-F 0 "#PWR0115" H 5150 1850 50  0001 C CNN
-F 1 "+5V" H 5165 2173 50  0000 C CNN
-F 2 "" H 5150 2000 50  0001 C CNN
-F 3 "" H 5150 2000 50  0001 C CNN
-	1    5150 2000
-	1    0    0    -1
-$EndComp
-$Comp
-L Connector:Screw_Terminal_01x03 J2
-U 1 1 5FA59775
-P 4300 2150
-F 0 "J2" H 4218 2367 50  0000 C CNN
-F 1 "Screw_Terminal_01x03" H 4218 2276 50  0000 C CNN
-F 2 "TerminalBlock_Phoenix:TerminalBlock_Phoenix_PT-1,5-2-3.5-H_1x02_P3.50mm_Horizontal" H 4300 2150 50  0001 C CNN
-F 3 "~" H 4300 2150 50  0001 C CNN
-	1    4300 2150
-	-1   0    0    -1
-$EndComp
-$Comp
-L power:GND #PWR0118
-U 1 1 5FA5A3CE
-P 4900 2250
-F 0 "#PWR0118" H 4900 2000 50  0001 C CNN
-F 1 "GND" H 4905 2077 50  0000 C CNN
-F 2 "" H 4900 2250 50  0001 C CNN
-F 3 "" H 4900 2250 50  0001 C CNN
-	1    4900 2250
-	1    0    0    -1
-$EndComp
 $Comp
 L Device:C_Small C2
@@
 	3200 3900 3150 3900
 Wire Wire Line
-	5150 2050 5150 2000
-Wire Wire Line
-	4500 2050 5150 2050
-Wire Wire Line
-	4900 2150 4900 2250
-Wire Wire Line
-	4500 2150 4900 2150
-Text Label 4600 2300 0    50   ~ 0
-PWM
-Wire Wire Line
-	4500 2250 4600 2250
-Wire Wire Line
-	4600 2250 4600 2300
+	4500 2150 4600 2150
+Wire Wire Line
+	4600 2150 4600 2250
+$Comp
+L power:GND #PWR0118
+U 1 1 5FA5A3CE
+P 4600 2250
+F 0 "#PWR0118" H 4600 2000 50  0001 C CNN
+F 1 "GND" H 4605 2077 50  0000 C CNN
+F 2 "" H 4600 2250 50  0001 C CNN
+F 3 "" H 4600 2250 50  0001 C CNN
+	1    4600 2250
+	1    0    0    -1
+$EndComp
+$Comp
+L Connector:Screw_Terminal_01x02 J2
+U 1 1 5FA59775
+P 4300 2050
+F 0 "J2" H 4218 2267 50  0000 C CNN
+F 1 "Screw_Terminal_01x02" H 4218 2176 50  0000 C CNN
+F 2 "TerminalBlock_Phoenix:TerminalBlock_Phoenix_PT-1,5-2-3.5-H_1x02_P3.50mm_Horizontal" H 4300 2050 50  0001 C CNN
+F 3 "~" H 4300 2050 50  0001 C CNN
+	1    4300 2050
+	-1   0    0    -1
+$EndComp
+Wire Wire Line
+	3050 4950 2900 4950
+Wire Wire Line
+	3050 5150 2900 5150
+Wire Wire Line
+	3050 5350 2900 5350
+Wire Wire Line
+	3050 5550 2900 5550
+Wire Wire Line
+	3050 5750 2900 5750
+Wire Wire Line
+	3050 5950 2900 5950
+Wire Wire Line
+	3650 5350 4150 5350
+Wire Wire Line
+	3650 5950 3650 5750
+Wire Wire Line
+	3650 5550 3650 5350
+Wire Wire Line
+	4350 5750 4400 5750
+Wire Wire Line
+	3650 5750 4150 5750
+$Comp
+L power:GND #PWR0133
+U 1 1 5FE58061
+P 4400 5750
+F 0 "#PWR0133" H 4400 5500 50  0001 C CNN
+F 1 "GND" V 4400 5650 50  0000 C CNN
+F 2 "" H 4400 5750 50  0001 C CNN
+F 3 "" H 4400 5750 50  0001 C CNN
+	1    4400 5750
+	0    -1   -1   0
+$EndComp
+$Comp
+L Device:R_Small R21
+U 1 1 5FE57D67
+P 4250 5750
+F 0 "R21" V 4250 5750 50  0000 C CNN
+F 1 "100k" V 4150 5550 50  0000 C CNN
+F 2 "Resistor_SMD:R_0603_1608Metric" H 4250 5750 50  0001 C CNN
+F 3 "~" H 4250 5750 50  0001 C CNN
+	1    4250 5750
+	0    1    1    0
+$EndComp
+Wire Wire Line
+	4350 5350 4400 5350
+Wire Wire Line
+	3650 5150 4150 5150
+Wire Wire Line
+	3650 4950 4150 4950
+Text Label 2900 5750 2    50   ~ 0
+DAA
+$Comp
+L power:GND #PWR0126
+U 1 1 5FDE9AF2
+P 4400 4950
+F 0 "#PWR0126" H 4400 4700 50  0001 C CNN
+F 1 "GND" V 4400 4850 50  0000 C CNN
+F 2 "" H 4400 4950 50  0001 C CNN
+F 3 "" H 4400 4950 50  0001 C CNN
+	1    4400 4950
+	0    -1   -1   0
+$EndComp
+$Comp
+L power:GND #PWR0127
+U 1 1 5FDEABE6
+P 4400 5150
+F 0 "#PWR0127" H 4400 4900 50  0001 C CNN
+F 1 "GND" V 4400 5050 50  0000 C CNN
+F 2 "" H 4400 5150 50  0001 C CNN
+F 3 "" H 4400 5150 50  0001 C CNN
+	1    4400 5150
+	0    -1   -1   0
+$EndComp
+$Comp
+L power:GND #PWR0128
+U 1 1 5FDFE31C
+P 4400 5350
+F 0 "#PWR0128" H 4400 5100 50  0001 C CNN
+F 1 "GND" V 4400 5250 50  0000 C CNN
+F 2 "" H 4400 5350 50  0001 C CNN
+F 3 "" H 4400 5350 50  0001 C CNN
+	1    4400 5350
+	0    -1   -1   0
+$EndComp
+$Comp
+L Device:R_Small R19
+U 1 1 5FD9157F
+P 4250 5150
+F 0 "R19" V 4250 5150 50  0000 C CNN
+F 1 "100k" V 4200 4950 50  0000 C CNN
+F 2 "Resistor_SMD:R_0603_1608Metric" H 4250 5150 50  0001 C CNN
+F 3 "~" H 4250 5150 50  0001 C CNN
+	1    4250 5150
+	0    1    1    0
+$EndComp
+$Comp
+L Device:R_Small R18
+U 1 1 5FD91E5A
+P 4250 4950
+F 0 "R18" V 4250 4950 50  0000 C CNN
+F 1 "100k" V 4150 4750 50  0000 C CNN
+F 2 "Resistor_SMD:R_0603_1608Metric" H 4250 4950 50  0001 C CNN
+F 3 "~" H 4250 4950 50  0001 C CNN
+	1    4250 4950
+	0    1    1    0
+$EndComp
+Wire Wire Line
+	4400 5150 4350 5150
+Wire Wire Line
+	4400 4950 4350 4950
+Text Label 2900 5950 2    50   ~ 0
+VINT
+Text Label 2900 5350 2    50   ~ 0
+CMTMOD
+Text Label 3700 5150 0    50   ~ 0
+FR
+Text Label 3700 4950 0    50   ~ 0
+BRKMOD
+Connection ~ 3650 5750
+Connection ~ 3650 5350
+$Comp
+L 1825057-5:1825057-5 SW1
+U 1 1 5FD8A0DD
+P 3350 5450
+F 0 "SW1" H 3350 6199 50  0000 C CNN
+F 1 "SW_DIP_x06" H 3350 6108 50  0000 C CNN
+F 2 "HS2_parts:DIP762W56P254L1772H585Q12" H 3350 5450 50  0001 C CNN
+F 3 "~" H 3350 5450 50  0001 C CNN
+	1    3350 5450
+	1    0    0    -1
+$EndComp
+$Comp
+L Device:R_Small R20
+U 1 1 5FD8CC05
+P 4250 5350
+F 0 "R20" V 4250 5350 50  0000 C CNN
+F 1 "100k" V 4200 5150 50  0000 C CNN
+F 2 "Resistor_SMD:R_0603_1608Metric" H 4250 5350 50  0001 C CNN
+F 3 "~" H 4250 5350 50  0001 C CNN
+	1    4250 5350
+	0    1    1    0
+$EndComp
+Text Label 2900 5550 2    50   ~ 0
+VINT
+Text Label 2900 5150 2    50   ~ 0
+VINT
+Text Label 2900 4950 2    50   ~ 0
+VINT
+$Comp
+L power:+5V #PWR0115
+U 1 1 5FA557E2
+P 5000 2050
+F 0 "#PWR0115" H 5000 1900 50  0001 C CNN
+F 1 "+5V" H 5015 2223 50  0000 C CNN
+F 2 "" H 5000 2050 50  0001 C CNN
+F 3 "" H 5000 2050 50  0001 C CNN
+	1    5000 2050
+	1    0    0    -1
+$EndComp
+$Comp
+L Connector:Conn_01x08_Male J3
+U 1 1 5FA7B2EB
+P 5700 5150
+F 0 "J3" H 5672 5124 50  0000 R CNN
+F 1 "Conn_01x08_Male" H 5672 5033 50  0000 R CNN
+F 2 "Connector_PinHeader_2.54mm:PinHeader_1x08_P2.54mm_Vertical" H 5700 5150 50  0001 C CNN
+F 3 "~" H 5700 5150 50  0001 C CNN
+	1    5700 5150
+	-1   0    0    -1
+$EndComp
+Wire Wire Line
+	4500 2050 5000 2050
 $EndSCHEMATC

Commit message: njoi
Parts:
- removed R18, R19, R20, R21: 100k, Resistor_SMD:R_0603_1608Metric, symbol Device:R_Small
- removed SW1: SW_DIP_x06, HS2_parts:DIP762W56P254L1772H585Q12, symbol 1825057-5:1825057-5
Connections:
- net +5V: now also J3.1 (Pin_1)
- net GND: now also J3.2 (Pin_2)
Changed lines of the file:
@@
 	-1   0    0    -1
 $EndComp
-Wire Wire Line
-	3050 4950 2900 4950
-Wire Wire Line
-	3050 5150 2900 5150
-Wire Wire Line
-	3050 5350 2900 5350
-Wire Wire Line
-	3050 5550 2900 5550
-Wire Wire Line
-	3050 5750 2900 5750
-Wire Wire Line
-	3050 5950 2900 5950
-Wire Wire Line
-	3650 5350 4150 5350
-Wire Wire Line
-	3650 5950 3650 5750
-Wire Wire Line
-	3650 5550 3650 5350
-Wire Wire Line
-	4350 5750 4400 5750
-Wire Wire Line
-	3650 5750 4150 5750
-$Comp
-L power:GND #PWR0133
-U 1 1 5FE58061
-P 4400 5750
-F 0 "#PWR0133" H 4400 5500 50  0001 C CNN
-F 1 "GND" V 4400 5650 50  0000 C CNN
-F 2 "" H 4400 5750 50  0001 C CNN
-F 3 "" H 4400 5750 50  0001 C CNN
-	1    4400 5750
-	0    -1   -1   0
-$EndComp
-$Comp
-L Device:R_Small R21
-U 1 1 5FE57D67
-P 4250 5750
-F 0 "R21" V 4250 5750 50  0000 C CNN
-F 1 "100k" V 4150 5550 50  0000 C CNN
-F 2 "Resistor_SMD:R_0603_1608Metric" H 4250 5750 50  0001 C CNN
-F 3 "~" H 4250 5750 50  0001 C CNN
-	1    4250 5750
-	0    1    1    0
-$EndComp
-Wire Wire Line
-	4350 5350 4400 5350
-Wire Wire Line
-	3650 5150 4150 5150
-Wire Wire Line
-	3650 4950 4150 4950
-Text Label 2900 5750 2    50   ~ 0
-DAA
-$Comp
-L power:GND #PWR0126
-U 1 1 5FDE9AF2
-P 4400 4950
-F 0 "#PWR0126" H 4400 4700 50  0001 C CNN
-F 1 "GND" V 4400 4850 50  0000 C CNN
-F 2 "" H 4400 4950 50  0001 C CNN
-F 3 "" H 4400 4950 50  0001 C CNN
-	1    4400 4950
-	0    -1   -1   0
-$EndComp
-$Comp
-L power:GND #PWR0127
-U 1 1 5FDEABE6
-P 4400 5150
-F 0 "#PWR0127" H 4400 4900 50  0001 C CNN
-F 1 "GND" V 4400 5050 50  0000 C CNN
-F 2 "" H 4400 5150 50  0001 C CNN
-F 3 "" H 4400 5150 50  0001 C CNN
-	1    4400 5150
-	0    -1   -1   0
-$EndComp
-$Comp
-L power:GND #PWR0128
-U 1 1 5FDFE31C
-P 4400 5350
-F 0 "#PWR0128" H 4400 5100 50  0001 C CNN
-F 1 "GND" V 4400 5250 50  0000 C CNN
-F 2 "" H 4400 5350 50  0001 C CNN
-F 3 "" H 4400 5350 50  0001 C CNN
-	1    4400 5350
-	0    -1   -1   0
-$EndComp
-$Comp
-L Device:R_Small R19
-U 1 1 5FD9157F
-P 4250 5150
-F 0 "R19" V 4250 5150 50  0000 C CNN
-F 1 "100k" V 4200 4950 50  0000 C CNN
-F 2 "Resistor_SMD:R_0603_1608Metric" H 4250 5150 50  0001 C CNN
-F 3 "~" H 4250 5150 50  0001 C CNN
-	1    4250 5150
-	0    1    1    0
-$EndComp
-$Comp
-L Device:R_Small R18
-U 1 1 5FD91E5A
-P 4250 4950
-F 0 "R18" V 4250 4950 50  0000 C CNN
-F 1 "100k" V 4150 4750 50  0000 C CNN
-F 2 "Resistor_SMD:R_0603_1608Metric" H 4250 4950 50  0001 C CNN
-F 3 "~" H 4250 4950 50  0001 C CNN
-	1    4250 4950
-	0    1    1    0
-$EndComp
-Wire Wire Line
-	4400 5150 4350 5150
-Wire Wire Line
-	4400 4950 4350 4950
-Text Label 2900 5950 2    50   ~ 0
-VINT
-Text Label 2900 5350 2    50   ~ 0
-CMTMOD
-Text Label 3700 5150 0    50   ~ 0
-FR
-Text Label 3700 4950 0    50   ~ 0
-BRKMOD
-Connection ~ 3650 5750
-Connection ~ 3650 5350
-$Comp
-L 1825057-5:1825057-5 SW1
-U 1 1 5FD8A0DD
-P 3350 5450
-F 0 "SW1" H 3350 6199 50  0000 C CNN
-F 1 "SW_DIP_x06" H 3350 6108 50  0000 C CNN
-F 2 "HS2_parts:DIP762W56P254L1772H585Q12" H 3350 5450 50  0001 C CNN
-F 3 "~" H 3350 5450 50  0001 C CNN
-	1    3350 5450
-	1    0    0    -1
-$EndComp
-$Comp
-L Device:R_Small R20
-U 1 1 5FD8CC05
-P 4250 5350
-F 0 "R20" V 4250 5350 50  0000 C CNN
-F 1 "100k" V 4200 5150 50  0000 C CNN
-F 2 "Resistor_SMD:R_0603_1608Metric" H 4250 5350 50  0001 C CNN
-F 3 "~" H 4250 5350 50  0001 C CNN
-	1    4250 5350
-	0    1    1    0
-$EndComp
-Text Label 2900 5550 2    50   ~ 0
-VINT
-Text Label 2900 5150 2    50   ~ 0
-VINT
-Text Label 2900 4950 2    50   ~ 0
-VINT
 $Comp
 L power:+5V #PWR0115
@@
 Wire Wire Line
 	4500 2050 5000 2050
+$Comp
+L power:+5V #PWR?
+U 1 1 6005D85A
+P 5350 4850
+F 0 "#PWR?" H 5350 4700 50  0001 C CNN
+F 1 "+5V" H 5365 5023 50  0000 C CNN
+F 2 "" H 5350 4850 50  0001 C CNN
+F 3 "" H 5350 4850 50  0001 C CNN
+	1    5350 4850
+	1    0    0    -1
+$EndComp
+$Comp
+L power:GND #PWR?
+U 1 1 6005E669
+P 5150 4950
+F 0 "#PWR?" H 5150 4700 50  0001 C CNN
+F 1 "GND" H 5155 4777 50  0000 C CNN
+F 2 "" H 5150 4950 50  0001 C CNN
+F 3 "" H 5150 4950 50  0001 C CNN
+	1    5150 4950
+	1    0    0    -1
+$EndComp
+Wire Wire Line
+	5500 4850 5350 4850
+Wire Wire Line
+	5500 4950 5150 4950
 $EndSCHEMATC

Commit message: Mostly finished PCB for ADC
Parts:
- J3: value Conn_01x08_Male -> Conn_01x03_Male; footprint Connector_PinHeader_2.54mm:PinHeader_1x08_P2.54mm_Vertical -> Connector_PinHeader_2.54mm:PinHeader_1x03_P2.54mm_Vertical; symbol Connector:Conn_01x08_Male -> Connector:Conn_01x03_Male
Connections:
- net PWM: now also J3.3 (Pin_3)
Changed lines of the file:
@@
 $EndComp
 $Comp
-L Connector:Conn_01x08_Male J3
+L Connector:Conn_01x03_Male J3
 U 1 1 5FA7B2EB
-P 5700 5150
-F 0 "J3" H 5672 5124 50  0000 R CNN
-F 1 "Conn_01x08_Male" H 5672 5033 50  0000 R CNN
-F 2 "Connector_PinHeader_2.54mm:PinHeader_1x08_P2.54mm_Vertical" H 5700 5150 50  0001 C CNN
-F 3 "~" H 5700 5150 50  0001 C CNN
-	1    5700 5150
+P 6400 2300
+F 0 "J3" H 6372 2274 50  0000 R CNN
+F 1 "Conn_01x03_Male" H 6350 2300 50  0000 R CNN
+F 2 "Connector_PinHeader_2.54mm:PinHeader_1x03_P2.54mm_Vertical" H 6400 2300 50  0001 C CNN
+F 3 "~" H 6400 2300 50  0001 C CNN
+	1    6400 2300
 	-1   0    0    -1
 $EndComp
@@
 L power:+5V #PWR?
 U 1 1 6005D85A
-P 5350 4850
-F 0 "#PWR?" H 5350 4700 50  0001 C CNN
-F 1 "+5V" H 5365 5023 50  0000 C CNN
-F 2 "" H 5350 4850 50  0001 C CNN
-F 3 "" H 5350 4850 50  0001 C CNN
-	1    5350 4850
+P 6050 2200
+F 0 "#PWR?" H 6050 2050 50  0001 C CNN
+F 1 "+5V" H 6065 2373 50  0000 C CNN
+F 2 "" H 6050 2200 50  0001 C CNN
+F 3 "" H 6050 2200 50  0001 C CNN
+	1    6050 2200
 	1    0    0    -1
 $EndComp
@@
 L power:GND #PWR?
 U 1 1 6005E669
-P 5150 4950
-F 0 "#PWR?" H 5150 4700 50  0001 C CNN
-F 1 "GND" H 5155 4777 50  0000 C CNN
-F 2 "" H 5150 4950 50  0001 C CNN
-F 3 "" H 5150 4950 50  0001 C CNN
-	1    5150 4950
+P 5850 2300
+F 0 "#PWR?" H 5850 2050 50  0001 C CNN
+F 1 "GND" H 5855 2127 50  0000 C CNN
+F 2 "" H 5850 2300 50  0001 C CNN
+F 3 "" H 5850 2300 50  0001 C CNN
+	1    5850 2300
 	1    0    0    -1
 $EndComp
 Wire Wire Line
-	5500 4850 5350 4850
+	6200 2200 6050 2200
 Wire Wire Line
-	5500 4950 5150 4950
+	6200 2300 5850 2300
+Text Label 6100 2400 2    50   ~ 0
+PWM
+Wire Wire Line
+	6200 2400 6100 2400
 $EndSCHEMATC
