File: Modular_single_driver_Regulator/Modular_single_driver_Regulator.sch (KiCad schematic (older format))
At the start: 39 parts, among them J1 Conn_02x02_Counter_Clockwise, J2 Screw_Terminal_01x02, J3 Conn_01x08_Male, SW1 SW_DIP_x06, U1 LTC6992-1 (Rev. D), U2 LM7805_TO220, U3 DRV10970

Commit message: Organized and renamed files
Parts:
- removed C10: 0.1u, Capacitor_SMD:C_0603_1608Metric, symbol Device:C_Small
- removed R1: 102k, Resistor_SMD:R_0603_1608Metric, symbol Device:R_Small
- removed R12: 619k, Resistor_SMD:R_0603_1608Metric, symbol Device:R_Small
- removed R13: 976k, Resistor_SMD:R_0603_1608Metric, symbol Device:R_Small
- removed R14: 50k, Resistor_SMD:R_0603_1608Metric, symbol Device:R_Small
- removed R15, R16: 1.25k, Resistor_SMD:R_0603_1608Metric, symbol Device:R_Small
- removed R17: 40k, Resistor_SMD:R_0603_1608Metric, symbol Device:R_Small
- removed RV1: 10k, HS2_parts:oldpot, symbol Device:R_POT
- removed U1: LTC6992-1 (Rev. D), Package_DFN_QFN:DFN-6-1EP_3x2mm_P0.5mm_EP1.65x1.35mm, symbol Timer:LTC6994xDCB-2
- added J4: Conn_01x03_Male, Connector_PinHeader_2.54mm:PinHeader_1x03_P2.54mm_Vertical, symbol Connector:Conn_01x03_Male
- R18, R19, R20, R21: value 10k -> 100k
Connections:
- net labels removed: IN
- wire segments 134 -> 115
Other:
- moved on the sheet: C1, C2, R18, R19, R20, R21

Commit message: yes
Parts:
- removed C5, C7, C8: 1u, Capacitor_SMD:C_0603_1608Metric, symbol Device:C_Small
- removed C6: 2.2u, Capacitor_SMD:C_0603_1608Metric, symbol Device:C_Small
- removed C9: 0.1u, Capacitor_SMD:C_0603_1608Metric, symbol Device:C_Small
- removed J1: Conn_02x02_Counter_Clockwise, Connector_PinHeader_2.54mm:PinHeader_2x02_P2.54mm_Vertical, symbol Connector_Generic:Conn_02x02_Counter_Clockwise
- removed J3: Conn_01x08_Male, Connector_PinHeader_2.54mm:PinHeader_1x08_P2.54mm_Vertical, symbol Connector:Conn_01x08_Male
- removed R10, R11, R9: 3.3k, Resistor_SMD:R_0603_1608Metric, symbol Device:R_Small
- removed R18, R19, R20, R21: 100k, Resistor_SMD:R_0603_1608Metric, symbol Device:R_Small
- removed R2, R3, R7, R8: 10k, Resistor_SMD:R_0603_1608Metric, symbol Device:R_Small
- removed R6: 200k, Resistor_SMD:R_0603_1608Metric, symbol Device:R_Small
- removed SW1: SW_DIP_x06, HS2_parts:DIP762W56P254L1772H585Q12, symbol 1825057-5:1825057-5
- removed U3: DRV10970, Package_SO:HTSSOP-24-1EP_4.4x7.8mm_P0.65mm_EP3.4x7.8mm_Mask2.4x4.68mm_ThermalVias, symbol HS2_Parts:DRV10970
- added J3: Conn_01x02_Male, Connector_PinHeader_2.54mm:PinHeader_1x02_P2.54mm_Vertical, symbol Connector:Conn_01x02_Male
- J2: renamed from J4; value Conn_01x03_Male -> Conn_01x02_Male; footprint Connector_PinHeader_2.54mm:PinHeader_1x03_P2.54mm_Vertical -> Connector_PinHeader_2.54mm:PinHeader_1x02_P2.54mm_Vertical; symbol Connector:Conn_01x03_Male -> Connector:Conn_01x02_Male
- renumbered C3 to C1, C4 to C2, C1 to C3, C2 to C4, D2 to D1, J2 to J1, R4 to R1, U2 to U1
Connections:
- net labels removed: BRKMOD, CMTMOD, DAA, FG, FR, HBIAS, HU, HV, HW, PWM, RD, VINT
- wire segments 115 -> 24
Other:
- note removed: "X7R"
- moved on the sheet: C3, C4
