File: Modular_single_driver_Regulator/Modular_single_driver_Regulator.kicad_pcb (KiCad board)
At the start: 2 copper layers, 10 parts, among them J1 Screw_Terminal_01x02, J2 Conn_01x02_Male, J3 Conn_01x02_Male, U1 LM7805_TO220

Commit message: yes
Other:
- board outline added: 35.3 x 13.2 mm
Changed lines of the file:
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@@
   (general
     (thickness 1.6)
-    (drawings 0)
+    (drawings 8)
     (tracks 24)
     (zones 0)
@@
   (page A4)
   (layers
-    (0 F.Cu signal hide)
-    (31 B.Cu signal hide)
+    (0 F.Cu signal)
+    (31 B.Cu signal)
     (32 B.Adhes user)
     (33 F.Adhes user)
@@
     (descr "TO-220-3, Vertical, RM 2.54mm, see https://www.vishay.com/docs/66542/to-220-1.pdf")
     (tags "TO-220-3 Vertical RM 2.54mm")
-    (fp_text reference U1 (at 2.54 -4.27) (layer F.SilkS)
+    (fp_text reference U1 (at 2.54 -2.032) (layer F.SilkS)
       (effects (font (size 1 1) (thickness 0.15)))
     )
@@
     )
   )
+  (gr_line (start 152.908 119.507) (end 152.908 109.093) (layer Edge.Cuts) (width 0.05))
+  (gr_line (start 186.817 120.904) (end 154.305 120.904) (layer Edge.Cuts) (width 0.05))
+  (gr_line (start 188.214 109.093) (end 188.214 119.507) (layer Edge.Cuts) (width 0.05))
+  (gr_line (start 154.305 107.696) (end 186.817 107.696) (layer Edge.Cuts) (width 0.05))
+  (gr_arc (start 154.305 109.093) (end 154.305 107.696) (angle -90) (layer Edge.Cuts) (width 0.05))
+  (gr_arc (start 154.305 119.507) (end 152.908 119.507) (angle -90) (layer Edge.Cuts) (width 0.05))
+  (gr_arc (start 186.817 119.507) (end 186.817 120.904) (angle -90) (layer Edge.Cuts) (width 0.05))
+  (gr_arc (start 186.817 109.093) (end 188.214 109.093) (angle -90) (layer Edge.Cuts) (width 0.05))
   (via (at 169.418 115.443) (size 0.8) (drill 0.4) (layers F.Cu B.Cu) (net 2))
   (via (at 164.465 114.3) (size 0.8) (drill 0.4) (layers F.Cu B.Cu) (net 2))

Commit message: some stuyff
Other:
- net class Default: trace_width 0.25 -> 0.2

Commit message: Yes they are
Parts:
- removed J2: Conn_01x02_Male, Connector_PinHeader_2.54mm:PinHeader_1x02_P2.54mm_Vertical
- moved J3 8.32 mm to (172.0, 111.8)
- moved J1 4.19 mm to (180.0, 113.2)
Connections:
- J3 pad 1: +5V -> GND
- J3 pad 2: GND -> +5V
Routing:
- net +12V: track 20.7 -> 28.3 mm
Other:
- board size 35.3 x 13.2 mm -> 31.5 x 13.2 mm
- board text added: "+12V"
- board text added: "+5V"
- board text added: "GND"
