File: Modular_MSP430/Modular_MSP430.sch (KiCad schematic (older format))
At the start: 18 parts

Commit message: Yes
Parts:
- added J?: Conn_01x03_Female, Connector_PinHeader_2.54mm:PinHeader_1x03_P2.54mm_Vertical, symbol Connector:Conn_01x03_Female
- C?: value .47u -> 0.47u
- U?: value LD1086V-DG -> LM3940
Connections:
- net +3V3: now also C?.1, U?.2 (OUT)
- net GND: now also J?.2 (Pin_2)
- net PWM: now also J?.3 (Pin_3)
- net +5V: now reaches C?.1, U?.3 (IN)
- net +5V: now also J?.1 (Pin_1)
Other:
- note added: "5V->3.3V Voltage Regulator"
- note added: "Basic Modular I/O"
- note added: "Driver Test Ports"
- moved on the sheet: C?, J?, U?
