File: Modular_single_driver_Driver/Modular_single_driver_Driver.sch (KiCad schematic (older format))
At the start: 30 parts, among them J1 Conn_02x02_Counter_Clockwise, J2 Screw_Terminal_01x02, J3 Conn_01x08_Male, J4 Conn_01x03_Male, SW1 SW_DIP_x06, U2 LM7805_TO220, U3 DRV10970

Commit message: More
Parts:
- removed C1, C2, C4: 0.1u, Capacitor_SMD:C_0603_1608Metric, symbol Device:C_Small
- removed C3: 0.33u, Capacitor_SMD:C_0603_1608Metric, symbol Device:C_Small
- removed D2: LED, LED_SMD:LED_1206_3216Metric, symbol Device:LED
- removed J2: Screw_Terminal_01x02, TerminalBlock_Phoenix:TerminalBlock_Phoenix_PT-1,5-2-3.5-H_1x02_P3.50mm_Horizontal, symbol Connector:Screw_Terminal_01x02
- removed R4: 510, Resistor_SMD:R_0603_1608Metric, symbol Device:R_Small
- removed U2: LM7805_TO220, Package_TO_SOT_THT:TO-220-3_Vertical, symbol Regulator_Linear:LM7805_TO220
Connections:
- net labels removed: +12V
- wire segments 115 -> 95
Changed lines of the file:
@@
 Text Label 6900 3250 2    50   ~ 0
 VINT
-$Comp
-L Device:R_Small R2
-U 1 1 5FA27BC3
-P 5750 3600
-F 0 "R2" V 5750 3600 50  0000 C CNN
-F 1 "10k" V 5850 3600 50  0000 C CNN
-F 2 "Resistor_SMD:R_0603_1608Metric" H 5750 3600 50  0001 C CNN
-F 3 "~" H 5750 3600 50  0001 C CNN
-	1    5750 3600
-	-1   0    0    1
-$EndComp
-$Comp
-L Device:R_Small R3
-U 1 1 5FA28A4B
-P 5750 3900
-F 0 "R3" V 5750 3900 50  0000 C CNN
-F 1 "10k" V 5850 3900 50  0000 C CNN
-F 2 "Resistor_SMD:R_0603_1608Metric" H 5750 3900 50  0001 C CNN
-F 3 "~" H 5750 3900 50  0001 C CNN
-	1    5750 3900
-	-1   0    0    1
-$EndComp
-$Comp
-L power:GND #PWR0111
-U 1 1 5FA28D4C
-P 5750 4000
-F 0 "#PWR0111" H 5750 3750 50  0001 C CNN
-F 1 "GND" H 5755 3827 50  0000 C CNN
-F 2 "" H 5750 4000 50  0001 C CNN
-F 3 "" H 5750 4000 50  0001 C CNN
-	1    5750 4000
-	1    0    0    -1
-$EndComp
-Wire Wire Line
-	5750 3500 5750 3450
-Text Label 5750 3450 1    50   ~ 0
-VINT
-Wire Wire Line
-	5750 3700 5750 3750
-Wire Wire Line
-	5750 3750 5700 3750
-Connection ~ 5750 3750
-Wire Wire Line
-	5750 3750 5750 3800
-Text Label 5700 3750 2    50   ~ 0
-HBIAS
 Wire Wire Line
 	7800 3650 7900 3650
@@
 Text Label 8000 3950 0    50   ~ 0
 HW
-$Comp
-L Regulator_Linear:LM7805_TO220 U2
-U 1 1 5FA49C5E
-P 5400 2050
-F 0 "U2" H 5400 2292 50  0000 C CNN
-F 1 "LM7805_TO220" H 5400 2201 50  0000 C CNN
-F 2 "Package_TO_SOT_THT:TO-220-3_Vertical" H 5400 2275 50  0001 C CIN
-F 3 "http://www.fairchildsemi.com/ds/LM/LM7805.pdf" H 5400 2000 50  0001 C CNN
-	1    5400 2050
-	1    0    0    -1
-$EndComp
-$Comp
-L power:GND #PWR0112
-U 1 1 5FA4A822
-P 5400 2450
-F 0 "#PWR0112" H 5400 2200 50  0001 C CNN
-F 1 "GND" H 5405 2277 50  0000 C CNN
-F 2 "" H 5400 2450 50  0001 C CNN
-F 3 "" H 5400 2450 50  0001 C CNN
-	1    5400 2450
-	1    0    0    -1
-$EndComp
-Wire Wire Line
-	5400 2350 5400 2450
-$Comp
-L Device:C_Small C3
-U 1 1 5FA4C83C
-P 4900 2300
-F 0 "C3" H 4992 2346 50  0000 L CNN
-F 1 "0.33u" H 4992 2255 50  0000 L CNN
-F 2 "Capacitor_SMD:C_0603_1608Metric" H 4900 2300 50  0001 C CNN
-F 3 "~" H 4900 2300 50  0001 C CNN
-	1    4900 2300
-	1    0    0    -1
-$EndComp
-$Comp
-L Device:C_Small C4
-U 1 1 5FA4CCCF
-P 5900 2350
-F 0 "C4" H 5992 2396 50  0000 L CNN
-F 1 "0.1u" H 5992 2305 50  0000 L CNN
-F 2 "Capacitor_SMD:C_0603_1608Metric" H 5900 2350 50  0001 C CNN
-F 3 "~" H 5900 2350 50  0001 C CNN
-	1    5900 2350
-	1    0    0    -1
-$EndComp
-$Comp
-L power:GND #PWR0114
-U 1 1 5FA4D458
-P 5900 2500
-F 0 "#PWR0114" H 5900 2250 50  0001 C CNN
-F 1 "GND" H 5905 2327 50  0000 C CNN
-F 2 "" H 5900 2500 50  0001 C CNN
-F 3 "" H 5900 2500 50  0001 C CNN
-	1    5900 2500
-	1    0    0    -1
-$EndComp
-Wire Wire Line
-	5900 2450 5900 2500
-Wire Wire Line
-	5100 2050 4900 2050
-Wire Wire Line
-	5700 2050 5900 2050
-Wire Wire Line
-	5900 2050 5900 2250
-$Comp
-L power:+5V #PWR0115
-U 1 1 5FA557E2
-P 5900 2050
-F 0 "#PWR0115" H 5900 1900 50  0001 C CNN
-F 1 "+5V" H 5915 2223 50  0000 C CNN
-F 2 "" H 5900 2050 50  0001 C CNN
-F 3 "" H 5900 2050 50  0001 C CNN
-	1    5900 2050
-	1    0    0    -1
-$EndComp
-Connection ~ 5900 2050
-$Comp
-L power:+12V #PWR0116
-U 1 1 5FA56096
-P 4900 2050
-F 0 "#PWR0116" H 4900 1900 50  0001 C CNN
-F 1 "+12V" H 4915 2223 50  0000 C CNN
-F 2 "" H 4900 2050 50  0001 C CNN
-F 3 "" H 4900 2050 50  0001 C CNN
-	1    4900 2050
-	1    0    0    -1
-$EndComp
-Connection ~ 4900 2050
-$Comp
-L Connector:Screw_Terminal_01x02 J2
-U 1 1 5FA59775
-P 4300 2050
-F 0 "J2" H 4218 2267 50  0000 C CNN
-F 1 "Screw_Terminal_01x02" H 4218 2176 50  0000 C CNN
-F 2 "TerminalBlock_Phoenix:TerminalBlock_Phoenix_PT-1,5-2-3.5-H_1x02_P3.50mm_Horizontal" H 4300 2050 50  0001 C CNN
-F 3 "~" H 4300 2050 50  0001 C CNN
-	1    4300 2050
-	-1   0    0    -1
-$EndComp
-$Comp
-L power:GND #PWR0118
-U 1 1 5FA5A3CE
-P 4600 2250
-F 0 "#PWR0118" H 4600 2000 50  0001 C CNN
-F 1 "GND" H 4605 2077 50  0000 C CNN
-F 2 "" H 4600 2250 50  0001 C CNN
-F 3 "" H 4600 2250 50  0001 C CNN
-	1    4600 2250
-	1    0    0    -1
-$EndComp
-Wire Wire Line
-	4500 2150 4600 2150
-Wire Wire Line
-	4600 2150 4600 2250
-Wire Wire Line
-	4900 2050 4500 2050
-$Comp
-L Device:C_Small C2
-U 1 1 5FA66D53
-P 4900 3550
-F 0 "C2" H 4808 3596 50  0000 R CNN
-F 1 "0.1u" H 4808 3505 50  0000 R CNN
-F 2 "Capacitor_SMD:C_0603_1608Metric" H 4900 3550 50  0001 C CNN
-F 3 "~" H 4900 3550 50  0001 C CNN
-	1    4900 3550
-	-1   0    0    -1
-$EndComp
-$Comp
-L Device:C_Small C1
-U 1 1 5FA67BE7
-P 4650 3550
-F 0 "C1" H 4558 3596 50  0000 R CNN
-F 1 "0.1u" H 4558 3505 50  0000 R CNN
-F 2 "Capacitor_SMD:C_0603_1608Metric" H 4650 3550 50  0001 C CNN
-F 3 "~" H 4650 3550 50  0001 C CNN
-	1    4650 3550
-	-1   0    0    -1
-$EndComp
-$Comp
-L power:GND #PWR0119
-U 1 1 5FA67EFE
-P 4800 3700
-F 0 "#PWR0119" H 4800 3450 50  0001 C CNN
-F 1 "GND" H 4805 3527 50  0000 C CNN
-F 2 "" H 4800 3700 50  0001 C CNN
-F 3 "" H 4800 3700 50  0001 C CNN
-	1    4800 3700
-	1    0    0    -1
-$EndComp
-Wire Wire Line
-	4650 3650 4650 3700
-Wire Wire Line
-	4650 3700 4800 3700
-Wire Wire Line
-	4900 3650 4900 3700
-Wire Wire Line
-	4900 3700 4800 3700
-Connection ~ 4800 3700
-Wire Wire Line
-	4650 3450 4650 3400
-Wire Wire Line
-	4650 3400 4750 3400
-Wire Wire Line
-	4900 3400 4900 3450
-$Comp
-L power:+5V #PWR0120
-U 1 1 5FA702C7
-P 4750 3400
-F 0 "#PWR0120" H 4750 3250 50  0001 C CNN
-F 1 "+5V" H 4765 3573 50  0000 C CNN
-F 2 "" H 4750 3400 50  0001 C CNN
-F 3 "" H 4750 3400 50  0001 C CNN
-	1    4750 3400
-	1    0    0    -1
-$EndComp
-Connection ~ 4750 3400
-Wire Wire Line
-	4750 3400 4900 3400
 Text Notes 6900 2550 0    50   ~ 0
 X7R
@@
 Text Label 9000 3700 2    50   ~ 0
 HW
-$Comp
-L Device:LED D2
-U 1 1 5FA9791C
-P 6250 2200
-F 0 "D2" V 6289 2082 50  0000 R CNN
-F 1 "LED" V 6198 2082 50  0000 R CNN
-F 2 "LED_SMD:LED_1206_3216Metric" H 6250 2200 50  0001 C CNN
-F 3 "~" H 6250 2200 50  0001 C CNN
-	1    6250 2200
-	0    -1   -1   0
-$EndComp
-Wire Wire Line
-	6250 2050 5900 2050
-$Comp
-L Device:R_Small R4
-U 1 1 5FA9C003
-P 6250 2500
-F 0 "R4" H 6309 2546 50  0000 L CNN
-F 1 "510" H 6309 2455 50  0000 L CNN
-F 2 "Resistor_SMD:R_0603_1608Metric" H 6250 2500 50  0001 C CNN
-F 3 "~" H 6250 2500 50  0001 C CNN
-	1    6250 2500
-	1    0    0    -1
-$EndComp
-Wire Wire Line
-	6250 2350 6250 2400
-$Comp
-L power:GND #PWR0123
-U 1 1 5FA9FF80
-P 6250 2650
-F 0 "#PWR0123" H 6250 2400 50  0001 C CNN
-F 1 "GND" H 6255 2477 50  0000 C CNN
-F 2 "" H 6250 2650 50  0001 C CNN
-F 3 "" H 6250 2650 50  0001 C CNN
-	1    6250 2650
-	1    0    0    -1
-$EndComp
-Wire Wire Line
-	6250 2600 6250 2650
-Wire Wire Line
-	4900 2050 4900 2200
-$Comp
-L power:GND #PWR0113
-U 1 1 5FB2AE6E
-P 4900 2400
-F 0 "#PWR0113" H 4900 2150 50  0001 C CNN
-F 1 "GND" H 4905 2227 50  0000 C CNN
-F 2 "" H 4900 2400 50  0001 C CNN
-F 3 "" H 4900 2400 50  0001 C CNN
-	1    4900 2400
-	1    0    0    -1
-$EndComp
 Wire Wire Line
 	6650 3000 6650 3050
@@
 Wire Wire Line
 	5250 5800 5100 5800
+Text Label 5700 3750 2    50   ~ 0
+HBIAS
+Wire Wire Line
+	5750 3750 5750 3800
+Connection ~ 5750 3750
+Wire Wire Line
+	5750 3750 5700 3750
+Wire Wire Line
+	5750 3700 5750 3750
+Text Label 5750 3450 1    50   ~ 0
+VINT
+Wire Wire Line
+	5750 3500 5750 3450
+$Comp
+L power:GND #PWR0111
+U 1 1 5FA28D4C
+P 5750 4000
+F 0 "#PWR0111" H 5750 3750 50  0001 C CNN
+F 1 "GND" H 5755 3827 50  0000 C CNN
+F 2 "" H 5750 4000 50  0001 C CNN
+F 3 "" H 5750 4000 50  0001 C CNN
+	1    5750 4000
+	1    0    0    -1
+$EndComp
+$Comp
+L Device:R_Small R3
+U 1 1 5FA28A4B
+P 5750 3900
+F 0 "R3" V 5750 3900 50  0000 C CNN
+F 1 "10k" V 5850 3900 50  0000 C CNN
+F 2 "Resistor_SMD:R_0603_1608Metric" H 5750 3900 50  0001 C CNN
+F 3 "~" H 5750 3900 50  0001 C CNN
+	1    5750 3900
+	-1   0    0    1
+$EndComp
+$Comp
+L Device:R_Small R2
+U 1 1 5FA27BC3
+P 5750 3600
+F 0 "R2" V 5750 3600 50  0000 C CNN
+F 1 "10k" V 5850 3600 50  0000 C CNN
+F 2 "Resistor_SMD:R_0603_1608Metric" H 5750 3600 50  0001 C CNN
+F 3 "~" H 5750 3600 50  0001 C CNN
+	1    5750 3600
+	-1   0    0    1
+$EndComp
 $EndSCHEMATC

Commit message: Updated connections and component values
- Updated component values to reflect those shown in the datasheet
- Connected HBIAS pins to each other
- Connected PowerPAD to ground plane
- Cleaned up traces
- Added some silkscreen labels to facilitate testing
Parts:
- C5: value 1u -> 10uF
- C6: value 2.2u -> 2.2uF
- C7, C8: value 1u -> 1uF
- C9: value 0.1u -> 0.1uF
- R6: value 200k -> 24k
- R7, R8: value 10k -> 3.3k
- SW1: symbol 1825057-5:1825057-5 -> Modular_single_driver_Driver-rescue:1825057-5-1825057-5
- U3: symbol HS2_Parts:DRV10970 -> Modular_single_driver_Driver-rescue:DRV10970-HS2_Parts
Changed lines of the file:
@@
 P 7650 2550
 F 0 "R8" V 7650 2550 50  0000 C CNN
-F 1 "10k" V 7750 2550 50  0000 C CNN
+F 1 "3.3k" V 7750 2550 50  0000 C CNN
 F 2 "Resistor_SMD:R_0603_1608Metric" H 7650 2550 50  0001 C CNN
 F 3 "~" H 7650 2550 50  0001 C CNN
@@
 P 7650 2300
 F 0 "R7" V 7550 2300 50  0000 C CNN
-F 1 "10k" V 7650 2300 50  0000 C CNN
+F 1 "3.3k" V 7650 2300 50  0000 C CNN
 F 2 "Resistor_SMD:R_0603_1608Metric" H 7650 2300 50  0001 C CNN
 F 3 "~" H 7650 2300 50  0001 C CNN
@@
 P 7200 2500
 F 0 "C9" V 6971 2500 50  0000 C CNN
-F 1 "0.1u" V 7062 2500 50  0000 C CNN
+F 1 "0.1uF" V 7062 2500 50  0000 C CNN
 F 2 "Capacitor_SMD:C_0603_1608Metric" H 7200 2500 50  0001 C CNN
 F 3 "~" H 7200 2500 50  0001 C CNN
@@
 P 6650 3250
 F 0 "C6" V 6600 3150 50  0000 C CNN
-F 1 "2.2u" V 6550 3300 50  0000 C CNN
+F 1 "2.2uF" V 6550 3300 50  0000 C CNN
 F 2 "Capacitor_SMD:C_0603_1608Metric" H 6650 3250 50  0001 C CNN
 F 3 "~" H 6650 3250 50  0001 C CNN
@@
 P 6450 3150
 F 0 "C5" V 6550 3200 50  0000 C CNN
-F 1 "1u" V 6500 3250 50  0000 C CNN
+F 1 "10uF" V 6500 3250 50  0000 C CNN
 F 2 "Capacitor_SMD:C_0603_1608Metric" H 6450 3150 50  0001 C CNN
 F 3 "~" H 6450 3150 50  0001 C CNN
@@
 P 6750 3050
 F 0 "C8" V 6800 2950 50  0000 C CNN
-F 1 "1u" V 6900 3050 50  0000 C CNN
+F 1 "1uF" V 6900 3050 50  0000 C CNN
 F 2 "Capacitor_SMD:C_0603_1608Metric" H 6750 3050 50  0001 C CNN
 F 3 "~" H 6750 3050 50  0001 C CNN
@@
 P 6800 4050
 F 0 "R6" V 6800 4050 50  0000 C CNN
-F 1 "200k" V 6850 4200 50  0000 C CNN
+F 1 "24k" V 6850 4200 50  0000 C CNN
 F 2 "Resistor_SMD:R_0603_1608Metric" H 6800 4050 50  0001 C CNN
 F 3 "~" H 6800 4050 50  0001 C CNN
@@
 $EndComp
 $Comp
-L 1825057-5:1825057-5 SW1
+L Modular_single_driver_Driver-rescue:1825057-5-1825057-5 SW1
 U 1 1 5FD8A0DD
 P 5550 5300
@@
 $EndComp
 $Comp
-L HS2_Parts:DRV10970 U3
+L Modular_single_driver_Driver-rescue:DRV10970-HS2_Parts U3
 U 1 1 5F9EAE81
 P 7300 3400
@@
 P 6650 3850
 F 0 "C7" V 6700 3950 50  0000 C CNN
-F 1 "1u" V 6750 3900 50  0000 C CNN
+F 1 "1uF" V 6750 3900 50  0000 C CNN
 F 2 "Capacitor_SMD:C_0603_1608Metric" H 6650 3850 50  0001 C CNN
 F 3 "~" H 6650 3850 50  0001 C CNN
